File: LFK2.kicad_sch (KiCad schematic)
At the start: 22 parts, among them J1 AVR-ISP-6, U1 ATmega32U4-M, U2 PRTR5V0U2X, Y1 Crystal_GND24_Small

Commit message: v2.0.0
Parts:
- C1, C2, C3, C4, C5, C6, C7, C8: footprint Capacitor_SMD:C_0805_2012Metric -> Capacitor_SMD:C_0402_1005Metric
- R1, R2, R3, R4, R5, R6: footprint Resistor_SMD:R_0805_2012Metric -> Resistor_SMD:R_0402_1005Metric

Commit message: v2.0.1
Left more room for traces (screws)
Parts:
- C8: footprint Capacitor_SMD:C_0402_1005Metric -> Capacitor_SMD:C_0603_1608Metric
Changed lines of the file:
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@@
       (effects (font (size 0.9 0.9)) (justify left))
     )
-    (property "Footprint" "Capacitor_SMD:C_0402_1005Metric" (id 2) (at 118.11 133.35 0)
+    (property "Footprint" "Capacitor_SMD:C_0603_1608Metric" (id 2) (at 118.11 133.35 0)
       (effects (font (size 1.27 1.27)) hide)
     )
@@
     )
     (path "/67d0ba3d-dbf9-447b-abe6-a71e8a0f11e5"
-      (reference "C8") (unit 1) (value "10u") (footprint "Capacitor_SMD:C_0402_1005Metric")
+      (reference "C8") (unit 1) (value "10u") (footprint "Capacitor_SMD:C_0603_1608Metric")
     )
     (path "/71755621-1f0d-4bdb-b18c-9e331608c358/34dcba5f-9b8b-4733-886a-cc4eef0f31ab"
