File: matrix.kicad_sch (KiCad schematic)
At the start: 130 parts, among them SW1 `~, SW10 9, SW11 0, SW12 -_, SW13 =+, SW14 BKSPC, SW15 DEL, SW16 TAB, SW17 Q, SW18 W, SW19 E, SW2 1, SW20 R, SW21 T, SW22 Y, SW23 U, SW24 I, SW25 O, SW26 P, SW27 [{, SW28 ]}, SW29 \|, SW3 2, SW30 HOME, SW31 CAPS, SW32 A, SW33 S, SW34 D, SW35 F, SW36 G, SW37 H, SW38 J, SW39 K, SW4 3, SW40 L, SW41 ;:, SW42 '", SW43 ENTER, SW44 LSHIFT, SW45 Z, SW46 X, SW47 C, SW48 V, SW49 B, SW5 4, SW50 N, SW51 M, SW52 ,<, SW53 .>, SW54 /?, SW55 RSHIFT, SW56 UP, SW57 LCTRL, SW58 LWIN, SW59 LALT, SW6 5, SW60 SPACE, SW61 RALT, SW62 FN, SW63 LEFT, SW64 DOWN, SW65 RIGHT, SW7 6, SW8 7, SW9 8

Commit message: v2.0.0
Parts:
- SW1, SW10, SW11, SW12, SW13, SW15, SW17, SW18, SW19, SW2, SW20, SW21, SW22, SW23, SW24, SW25, SW26, SW27, SW28, SW3, SW30, SW32, SW33, SW34, SW35, SW36, SW37, SW38, SW39, SW4, SW40, SW41, SW42, SW45, SW46, SW47, SW48, SW49, SW5, SW50, SW51, SW52, SW53, SW54, SW56, SW6, SW63, SW64, SW65, SW7, SW8, SW9: footprint MX_Only:MXOnly-1U -> MX_Only:MXOnly-1U-Hotswap
- SW14: footprint MX_Only:MXOnly-2U -> MX_Only:MXOnly-2U-Hotswap
- SW16, SW29: footprint MX_Only:MXOnly-1.5U -> MX_Only:MXOnly-1.5U-Hotswap
- SW31: footprint MX_Only:MXOnly-1.75U -> MX_Only:MXOnly-1.75U-Hotswap-Double
- SW43, SW44: footprint MX_Only:MXOnly-2.25U -> MX_Only:MXOnly-2.25U-Hotswap
- SW55: footprint MX_Only:MXOnly-1.75U -> MX_Only:MXOnly-1.75U-Hotswap
- SW57, SW59, SW62: footprint MX_Only:MXOnly-1.25U -> MX_Only:MXOnly-1.5U-Hotswap-Double
- SW58, SW61: footprint MX_Only:MXOnly-1.25U -> MX_Only:MXOnly-1.25U-Hotswap
- SW60: footprint MX_Only:MXOnly-6.25U-ReversedStabilizers -> MX_Only:MXOnly-6.25U-Hotswap-RS-Double

Commit message: v2.1.1
Tsangan WK and Small Fixes
Parts:
- added SW66: TLCTRL, MX_Only:MXOnly-1.5U-Hotswap, symbol Switch:SW_Push
- added SW67: TLALT, MX_Only:MXOnly-1.5U-Hotswap, symbol Switch:SW_Push
- added SW68: TSPACE, MX_Only:MXOnly-7U-Hotswap, symbol Switch:SW_Push
- added SW69: TRALT, MX_Only:MXOnly-1.5U-Hotswap, symbol Switch:SW_Push
- added SW70: TLWIN, MX_Only:MXOnly-1U-Hotswap, symbol Switch:SW_Push
- SW31: footprint MX_Only:MXOnly-1.75U-Hotswap-Double -> MX_Only:MXOnly-1.75U-Hotswap
- SW57, SW59, SW62: footprint MX_Only:MXOnly-1.5U-Hotswap-Double -> MX_Only:MXOnly-1.25U-Hotswap
- SW60: footprint MX_Only:MXOnly-6.25U-Hotswap-RS-Double -> MX_Only:MXOnly-6.25U-Hotswap-ReversedStabilizers
Connections:
- net col0: now also SW66.1
- net col1: now also SW70.1
- net col11: now also SW69.1
- net col2: now also SW67.1
- net col5: now also SW68.1
- net at D59.2 (A), SW59.2: now also SW67.2
- net at D62.2 (A), SW62.2: now also SW69.2
- net at D58.2 (A), SW58.2: now also SW70.2
- net at D57.2 (A), SW57.2: now also SW66.2
- net at D60.2 (A), SW60.2: now also SW68.2
Other:
- moved on the sheet: D58, SW58
